File: hardware/mega-shield/xc2064-mega-shield.kicad_pcb (KiCad board)
At the start: 4 copper layers, 101.6 x 53.3 mm, 80 parts, among them J1 Conn_01x08, J2 Conn_01x10, J3 Conn_01x08, J4 Conn_01x08, J5 Conn_01x08, J6 Conn_01x08, J7 Conn_02x18, J8 Conn_01x02, SW1 SW_Push, U1 XC2064-PC68, U2 TPS22917DBV, U3 INA226, U4 74HCT541, Y2 4MHz

Commit message: Update Shield
Routing:
- net VCC_FPGA: track 158.0 -> 147.5 mm, vias 6 -> 4
